File: pcb/fissure/fissure.kicad_pcb (KiCad board)
At the start: 2 copper layers, 217 x 154.7 mm, 202 parts, among them J1 debug-port, J11 Conn_01x12_Socket, J12 Conn_01x12_Pin, J16 Conn_01x12_Pin, J17 Conn_01x12_Socket, J2 USB_C_Receptacle_USB2.0, J3 Conn_01x12_Pin, J4 Conn_01x12_Pin, J5 cirque-trackpad, J6 Conn_01x12_Socket, J7 Conn_01x12_Socket, J8 USB_C_Receptacle_USB2.0, J9 debug-port, K1 diode-choc, K10 diode-choc, K11 diode-choc, K12 diode-choc, K13 diode-choc, K14 diode-choc, K15 diode-choc, K16 diode-choc, K17 diode-choc, K18 diode-choc, K19 diode-choc, K2 diode-choc, K20 diode-choc, K21 diode-choc, K22 diode-choc, K23 diode-choc, K24 diode-choc, K25 diode-choc, K26 diode-choc, K27 diode-choc, K28 diode-choc, K29 diode-choc, K3 diode-choc, K30 diode-choc, K31 diode-choc, K32 diode-choc, K33 diode-choc, K34 diode-choc, K35 diode-choc, K36 diode-choc, K37 diode-choc, K38 diode-choc, K39 diode-choc, K4 diode-choc, K40 diode-choc, K5 diode-choc, K6 diode-choc, K7 diode-choc, K8 diode-choc, K9 diode-choc, Q1 AO3400A, Q2 AO3400A, SW1 SW_Push, SW2 SW_Push, SW3 SW_SPDT, SW4 SW_SPDT, U1 e73-2gm08s1c, U10 W25Q128JVS, U11 DW01A, U12 e73-2gm08s1c, U13 IS31FL3729, U14 DW01A, U15 FS8205, U16 FS8205, U2 W25Q128JVS, U3 BQ24075, U4 TLV62568DBV, U5 PMW3610, U6 IS31FL3729, U7 SRV05-4, U8 SRV05-4, U9 BQ24075

Commit message: break out points
Parts:
- added TP1: CS, TestPoint:TestPoint_THTPad_D1.0mm_Drill0.5mm, F.Cu at (185.3, 90.5)
- added TP2: SCLK, TestPoint:TestPoint_THTPad_D1.0mm_Drill0.5mm, F.Cu at (179.3, 90.5)
- added TP3: MISO, TestPoint:TestPoint_THTPad_D1.0mm_Drill0.5mm, F.Cu at (181.3, 90.5)
- added TP4: MOSI, TestPoint:TestPoint_THTPad_D1.0mm_Drill0.5mm, F.Cu at (183.3, 90.5)
- added TP5: SDA, TestPoint:TestPoint_THTPad_D1.0mm_Drill0.5mm, F.Cu at (189.3, 90.5)
- added TP6: SCL, TestPoint:TestPoint_THTPad_D1.0mm_Drill0.5mm, F.Cu at (187.3, 90.5)
- added TP7: 3V3, TestPoint:TestPoint_THTPad_D1.0mm_Drill0.5mm, F.Cu at (179.9, 88.2)
- added TP8: GND, TestPoint:TestPoint_THTPad_D1.0mm_Drill0.5mm, F.Cu at (191.7, 88.7)
Connections:
- U1 pad 16: unconnected-(U1-P0.08-Pad16) -> R_CS3
Routing:
- net R_CS3: track 0.00 -> 103.4 mm, vias 0 -> 7
- net R_SCL: track 13.7 -> 91.2 mm, vias 2 -> 4
- net R_SDA: track 11.6 -> 84.3 mm, vias 2 -> 4
- net R_MISO: track 115.2 -> 118.5 mm, vias 3 -> 4
- net R_SCLK: track 129.7 -> 132.6 mm, vias 3 -> 4
- net R_ROW0: track 165.8 -> 163.1 mm, vias 9 -> 11
- net Net-(D12C-A): track 57.2 -> 55.8 mm
- net L_GND: track 257.2 -> 258.5 mm, vias 162 -> 161
- net Net-(D11D-A): track 34.3 -> 33.3 mm
- net R_MOSI: track 131.7 -> 132.6 mm
- net R_COL0: track 24.5 -> 23.6 mm
- net MOTION: track 89.9 -> 90.7 mm
- net MOUSE_~{RST}: track 88.4 -> 89.2 mm
- net /thumb+led_r/A1: track 139.8 -> 140.6 mm
- net +1V8: track 37.2 -> 36.6 mm
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
Commit message: v3.3 production
Parts:
- added QR*****: github, fissure:github, B.Cu at (114.8, -11.0)
- added REF**: mousebites, misc:mousebites, F.Cu at (156.5, 32.0)
- added REF**: mousebites, misc:mousebites, F.Cu at (137.5, 74.5)
- added REF**: mousebites, misc:mousebites, F.Cu at (134.5, -7.50)
- added REF**: mousebites, misc:mousebites, F.Cu at (114.0, 27.0)
- added REF**: jlc-tooling-hole, misc:jlc-tooling-hole, F.Cu at (139.5, -18.5)
- added REF**: mousebites, misc:mousebites, F.Cu at (137.5, 55.5)
- added REF**: mousebites, misc:mousebites, F.Cu at (137.5, 11.5)
- added REF**: mousebites, misc:mousebites, F.Cu at (161.5, 35.0)
- added REF**: mousebites, misc:mousebites, F.Cu at (224.0, 32.0)
- added REF**: mousebites, misc:mousebites, F.Cu at (156.5, 35.0)
- added REF**: mousebites, misc:mousebites, F.Cu at (125.5, -13.0)
- added REF**: mousebites, misc:mousebites, F.Cu at (161.5, 32.0)
- added REF**: mousebites, misc:mousebites, F.Cu at (219.0, 32.0)
- added REF**: mousebites, misc:mousebites, F.Cu at (122.5, -13.0)
- added REF**: jlc-tooling-hole, misc:jlc-tooling-hole, F.Cu at (139.5, 85.5)
- added REF**: mousebites, misc:mousebites, F.Cu at (125.5, 80.0)
- added REF**: mousebites, misc:mousebites, F.Cu at (219.0, 35.0)
- added REF**: mousebites, misc:mousebites, F.Cu at (137.5, -7.50)
- added REF**: jlc-tooling-hole, misc:jlc-tooling-hole, F.Cu at (222.0, -21.5)
- added REF**: mousebites, misc:mousebites, F.Cu at (114.0, 40.0)
- added REF**: mousebites, misc:mousebites, F.Cu at (134.5, 55.5)
- added REF**: mousebites, misc:mousebites, F.Cu at (137.5, 42.5)
- added REF**: mousebites, misc:mousebites, F.Cu at (224.0, 35.0)
- added REF**: jlc-tooling-hole, misc:jlc-tooling-hole, F.Cu at (195.5, 119.5)
- added REF**: mousebites, misc:mousebites, F.Cu at (134.5, 11.5)
- added REF**: mousebites, misc:mousebites, F.Cu at (137.5, 24.5)
- added REF**: mousebites, misc:mousebites, F.Cu at (122.5, 80.0)
- added REF**: mousebites, misc:mousebites, F.Cu at (134.5, 74.5)
- D10, D11, D12, D3, D4, D5, D6, D7, D8, D9: value ~ -> 1SS309
- moved K20 240.2 mm to (148.2, -40.5), turned to -90 degrees
- moved LED20 236.3 mm to (143.5, -40.5), turned to -90 degrees
- moved K19 232.5 mm to (133.2, -42.5), turned to -90 degrees
- moved K18 230.6 mm to (118.2, -45.5), turned to -90 degrees
- moved LED19 229.7 mm to (128.5, -42.5), turned to -90 degrees
- moved LED18 228.9 mm to (113.5, -45.5), turned to -90 degrees
- moved K17 225.4 mm to (227.5, -16.5), turned to 0 degrees
- moved LED17 221.4 mm to (227.5, -11.8), turned to 180 degrees
- moved K11 215.6 mm to (212.5, -31.5), turned to 0 degrees
- moved D3 213.9 mm to (230.7, 9.30), turned to 90 degrees
- moved K16 213.8 mm to (227.5, -1.50), turned to 0 degrees
- moved LED16 210.9 mm to (227.5, 3.20), turned to 180 degrees
- moved LED11 210.1 mm to (212.5, -26.8), turned to 180 degrees
- moved D4 207.3 mm to (227.3, 9.30), turned to 90 degrees
- moved U2 202.4 mm to (227.6, 28.5), turned to 180 degrees
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- gave numbers to parts that had none: 6
Routing:
- net L_GND: track 258.5 -> 243.6 mm, vias 161 -> 163
- net L_SWD: track 74.3 -> 75.1 mm
- net L_3V3: vias 4 -> 5
Other:
- board size 217 x 154.7 mm -> 131.5 x 184.4 mm
